Commit message: collect calibration data

File: ur_description/urdf/common.gazebo.xacro (robot description, xacro)
@@ -3,6 +3,6 @@
   <gazebo>
     <plugin name="gazebo_ros_control" filename="libgazebo_ros_control.so">
-      <robotNamespace>/ur5</robotNamespace>
-      <robotSimType>gazebo_ros_control/DefaultRobotHWSim</robotSimType>
+      <!-- <robotNamespace>/ur5</robotNamespace> -->
+      <!-- <robotSimType>gazebo_ros_control/DefaultRobotHWSim</robotSimType> -->
     </plugin>
 <!--

File: ur_description/urdf/ur5_joint_limited_robot.urdf.xacro (robot description, xacro)
@@ -8,7 +8,9 @@
   <!-- ur5 -->
   <xacro:include filename="$(find ur_description)/urdf/ur5.urdf.xacro" />
+  <!-- kinect camera -->
+  <xacro:include filename="$(find hector_sensors_description)/urdf/kinect_camera.urdf.xacro" />
   <!-- photoneo camera -->
-  <xacro:include filename="$(find phoxi_camera)/urdf/PhoXi3Dscanner_values.xacro"/> <!--Scanner values-->
-  <xacro:include filename="$(find phoxi_camera)/urdf/PhoXi3Dscanner_macro.xacro"/>  <!--Scanner macro-->
+  <!-- <xacro:include filename="$(find phoxi_camera)/urdf/PhoXi3Dscanner_values.xacro"/>  -->
+  <!-- <xacro:include filename="$(find phoxi_camera)/urdf/PhoXi3Dscanner_macro.xacro"/>   -->
   <!-- workplatform-->
   <xacro:include filename="$(find ur_description)/urdf/platform.urdf.xacro" />
@@ -27,5 +29,5 @@
   <joint name="world_joint" type="fixed">
     <parent link="world" />
-    <child link = "box" />
+    <child link = "base_link" />
     <origin xyz="0.0 0.0 0.0" rpy="0.0 0.0 0.0" />
   </joint>
@@ -33,12 +35,33 @@
   <!-- <xacro:rg2 prefix="${prefix}"/> -->
   <!-- photoneo camare -->
-  <xacro:PhoXi3Dscanner scanner_parent = "base_link" scanner_name = "PhoXi3Dscanner" sensor_parent = "PhoXi3Dscanner" sensor_name = "PhoXi3Dscanner_sensor" >
-      <origin xyz="0.075 0.928 0.535" rpy="${pi-pi/6-pi/50} 0.02 0" /> <!--PhoXi3Dscanner origin-->
-      <xacro:PhoXi3DscannerS_default_sensor_origin /> <!--Extrinsic calibration data-->
-      <xacro:PhoXi3DscannerS_meshes /> <!--meshes-->
-  </xacro:PhoXi3Dscanner>
-  <!-- workplatform -->
-  <xacro:boxbase child="base_link" >
-    <origin xyz="0.0 0.0 ${boxz}" rpy="0.0 0.0 0.0"/>
-  </xacro:boxbase>
+  <!-- <xacro:PhoXi3Dscanner scanner_parent = "base_link" scanner_name = "PhoXi3Dscanner" sensor_parent = "PhoXi3Dscanner" sensor_name = "PhoXi3Dscanner_sensor" >
+      <origin xyz="0.075 0.928 0.535" rpy="${pi-pi/6-pi/50} 0.02 0" />
+      <xacro:PhoXi3DscannerS_default_sensor_origin />
+      <xacro:PhoXi3DscannerS_meshes />
+  </xacro:PhoXi3Dscanner> -->
+  <!-- kinect camare -->
+  <xacro:kinect_camera parent="base_link" name="kinect">
+    <origin xyz="0.6 0 1" rpy="0.0 ${pi/2} 0"/>
+  </xacro:kinect_camera>
+  <!-- walls -->
+  <link name="wall">
+    <visual>
+      <geometry>
+        <box size="2 2 0.001"/>
+      </geometry>
+      <material name="gray"/>
+      <origin xyz="0 0 0.0005" rpy="0 -0 0"/>
+    </visual>
+    <collision>
+      <geometry>
+        <box size="2 2 0.001"/>
+      </geometry>
+    </collision>
+    <xacro:default_inertial mass="0.1"/>
+  </link>
+  <joint name="world_wall_joint" type="fixed">
+    <parent link="world" />
+    <child link = "wall" />
+    <origin xyz="-0.0 0.0 -0.05" rpy="0.0 0.0 0.0" />
+  </joint>
 </robot>
